File: kicad/m1s-fpga-playground/m1s-fpga-playground.kicad_sch (KiCad schematic)
At the start: 59 parts, among them J1 Conn_02x20_Odd_Even, J2 Conn_02x07_Odd_Even, J7 Pin Header, SW101 KMR2, SW102 KMR2, SW103 KMR2, SW104 KMR2, SW105 KMR2, U1 TLV71312PDBV, U106 AS4C32M8SA, U3 W25Q16JLSSIG, U4 ICE40HX4K-TQ144, X1 ECS-2520MV-xxx-xx

Commit message: Swapped pins 128 and 129 - PLL conflict
Connections:
- net 128: now also U106.53 (DQ7); no longer R1.1
- net 129: now also R1.1; no longer U106.53 (DQ7)
